File: Cyndel.kicad_pcb (KiCad board)
At the start: 2 copper layers, 0 parts

Commit message: add LED network and power
Parts:
- added D1, D10, D11, D12, D13, D14, D15, D16, D17, D18, D19, D2, D20, D3, D4, D5, D6, D7, D8, D9: LED_RABG, LEDs:LED_Cree-PLCC4, F.Cu at (148.5, 105.0)
- added R1, R10, R11, R12, R13, R14, R15, R16, R17, R18, R19, R2, R20, R21, R22, R23, R24, R25, R26, R27, R28, R29, R3, R30, R31, R32, R33, R34, R35, R36, R37, R38, R39, R4, R40, R41, R42, R43, R44, R45, R46, R47, R48, R49, R5, R50, R51, R52, R53, R54, R55, R56, R57, R58, R59, R6, R60, R7, R8, R9: 220R, Resistors_SMD:R_0603, F.Cu at (148.5, 105.0)
